File: projector-board/process_control.kicad_sch (KiCad schematic)
At the start: 1 part, among them U2 DLPC1438

Commit message: More projector power supply design
Parts:
- U2: Digikey (none) -> ORDER FROM TI
Other:
- company: (none) -> MICHIGAN TECH OPEN SOURCE HARDWARE ENTERPRISE
- title: (none) -> LITHO_PROJECTOR
Changed lines of the file:
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@@
 	(generator_version "10.0")
 	(paper "USLedger")
+	(title_block
+		(title "LITHO_PROJECTOR")
+		(date "2026-10-11")
+		(rev "v1")
+		(company "MICHIGAN TECH OPEN SOURCE HARDWARE ENTERPRISE")
+		(comment 1 "Author: Andrew Kroll <ajkroll@mtu.edu>")
+	)
 	(symbol
 		(lib_id "litho:DLPC1438")
@@
 				)
 				(justify left top)
+			)
+		)
+		(property "Digikey" "ORDER FROM TI"
+			(at 218.44 72.39 0)
+			(hide yes)
+			(show_name no)
+			(do_not_autoplace no)
+			(effects
+				(font
+					(size 1.27 1.27)
+				)
 			)
 		)
@@
 			)
 		)
+		(property "Digikey" "ORDER FROM TI"
+			(at 127 86.36 0)
+			(hide yes)
+			(show_name no)
+			(do_not_autoplace no)
+			(effects
+				(font
+					(size 1.27 1.27)
+				)
+			)
+		)
 		(pin "N10"
 		)
@@
 			)
 		)
+		(property "Digikey" "ORDER FROM TI"
+			(at 125.73 180.34 0)
+			(hide yes)
+			(show_name no)
+			(do_not_autoplace no)
+			(effects
+				(font
+					(size 1.27 1.27)
+				)
+			)
+		)
 		(pin "N10"
 		)
@@
 			)
 		)
+		(property "Digikey" "ORDER FROM TI"
+			(at 247.65 184.15 0)
+			(hide yes)
+			(show_name no)
+			(do_not_autoplace no)
+			(effects
+				(font
+					(size 1.27 1.27)
+				)
+			)
+		)
 		(pin "N10"
 		)
@@
 			)
 		)
+		(property "Digikey" "ORDER FROM TI"
+			(at 114.3 118.11 0)
+			(hide yes)
+			(show_name no)
+			(do_not_autoplace no)
+			(effects
+				(font
+					(size 1.27 1.27)
+				)
+			)
+		)

Commit message: Finish SPI bus
Other:
- moved on the sheet: U2B, U2C
Changed lines of the file:
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@@
 	(symbol
 		(lib_id "litho:DLPC1438")
-		(at 218.44 72.39 0)
+		(at 218.44 85.09 0)
 		(unit 2)
 		(body_style 1)
@@
 		(fields_autoplaced yes)
 		(property "Reference" "U2"
-			(at 218.44 111.76 0)
+			(at 218.44 124.46 0)
 			(show_name no)
 			(do_not_autoplace no)
@@
 		)
 		(property "Value" "DLPC1438"
-			(at 218.44 114.3 0)
+			(at 218.44 127 0)
 			(show_name no)
 			(do_not_autoplace no)
@@
 		)
 		(property "Footprint" "litho:NFBGA201"
-			(at 200.66 171.45 0)
+			(at 200.66 184.15 0)
 			(hide yes)
 			(show_name no)
@@
 		)
 		(property "Datasheet" "https://www.ti.com/product/DLPC1438"
-			(at 200.66 174.955 0)
+			(at 200.66 187.655 0)
 			(hide yes)
 			(show_name no)
@@
 		)
 		(property "Description" "Display Drivers & Controllers DLP controller for DLP300S and DLP301S digital micromirror devices (DMDs)"
-			(at 210.82 164.795 0)
+			(at 210.82 177.495 0)
 			(hide yes)
 			(show_name no)
@@
 		)
 		(property "Height" "1"
-			(at 96.52 455.88 0)
+			(at 96.52 468.58 0)
 			(hide yes)
 			(show_name no)
@@
 		)
 		(property "Digikey" "ORDER FROM TI"
-			(at 218.44 72.39 0)
+			(at 218.44 85.09 0)
 			(hide yes)
 			(show_name no)
@@
 	(symbol
 		(lib_id "litho:DLPC1438")
-		(at 127 86.36 0)
+		(at 124.46 71.12 0)
 		(unit 3)
 		(body_style 1)
@@
 		(fields_autoplaced yes)
 		(property "Reference" "U2"
-			(at 140.97 86.9949 0)
+			(at 138.43 71.7549 0)
 			(show_name no)
 			(do_not_autoplace no)
@@
 		)
 		(property "Value" "DLPC1438"
-			(at 140.97 89.5349 0)
+			(at 138.43 74.2949 0)
 			(show_name no)
 			(do_not_autoplace no)
@@
 		)
 		(property "Footprint" "litho:NFBGA201"
-			(at 109.22 185.42 0)
+			(at 106.68 170.18 0)
 			(hide yes)
 			(show_name no)
@@
 		)
 		(property "Datasheet" "https://www.ti.com/product/DLPC1438"
-			(at 109.22 188.925 0)
+			(at 106.68 173.685 0)
 			(hide yes)
 			(show_name no)
@@
 		)
 		(property "Description" "Display Drivers & Controllers DLP controller for DLP300S and DLP301S digital micromirror devices (DMDs)"
-			(at 119.38 178.765 0)
+			(at 116.84 163.525 0)
 			(hide yes)
 			(show_name no)
@@
 		)
 		(property "Height" "1"
-			(at 5.08 469.85 0)
+			(at 2.54 454.61 0)
 			(hide yes)
 			(show_name no)
@@
 		)
 		(property "Digikey" "ORDER FROM TI"
-			(at 127 86.36 0)
-			(hide yes)
-			(show_name no)
+			(at 124.46 71.12 0)
+			(hide yes)
+			(show_name no)
