File: projector-board/projector.kicad_sch (KiCad schematic)
At the start: 0 parts

Commit message: Add DMD PMIC Symbol
From Ultralibrarian
Parts:
- added U1: DLPA2000DYFFR, YFF56_TEX, symbol litho:DLPA2000DYFFR
Changed lines of the file:
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@@
 	(generator "eeschema")
 	(generator_version "10.0")
-	(paper "A4")
+	(paper "USLedger")
+	(symbol
+		(lib_id "litho:DLPA2000DYFFR")
+		(at 185.42 92.71 0)
+		(unit 1)
+		(body_style 1)
+		(exclude_from_sim no)
+		(in_bom yes)
+		(on_board yes)
+		(in_pos_files yes)
+		(dnp no)
+		(fields_autoplaced yes)
+		(property "Reference" "U1"
+			(at 215.9 82.55 0)
+			(show_name no)
+			(do_not_autoplace no)
+			(effects
+				(font
+					(size 1.524 1.524)
+				)
+			)
+		)
+		(property "Value" "DLPA2000DYFFR"
+			(at 215.9 85.09 0)
+			(show_name no)
+			(do_not_autoplace no)
+			(effects
+				(font
+					(size 1.524 1.524)
+				)
+			)
+		)
+		(property "Footprint" "YFF56_TEX"
+			(at 185.42 92.71 0)
+			(hide yes)
+			(show_name no)
+			(do_not_autoplace no)
+			(effects
+				(font
+					(size 1.27 1.27)
+					(italic yes)
+				)
+			)
+		)
+		(property "Datasheet" "https://www.ti.com/lit/gpn/dlpa2000"
+			(at 185.42 92.71 0)
+			(hide yes)
+			(show_name no)
+			(do_not_autoplace no)
+			(effects
+				(font
+					(size 1.27 1.27)
+					(italic yes)
+				)
+			)
+		)
+		(property "Description" ""
+			(at 185.42 92.71 0)
+			(hide yes)
+			(show_name no)
+			(do_not_autoplace no)
+			(effects
+				(font
+					(size 1.27 1.27)
+				)
+			)
+		)
+		(pin "H5"
+		)
+		(pin "C4"
+		)
+		(pin "F5"
+		)
+		(pin "G3"
+		)
+		(pin "A2"
+		)
+		(pin "E3"
+		)
+		(pin "F7"
+		)
+		(pin "H3"
+		)
+		(pin "D7"
+		)
+		(pin "F1"
+		)
+		(pin "G5"
+		)
+		(pin "D5"
+		)
+		(pin "H4"
+		)
+		(pin "D2"
+		)
+		(pin "E6"
+		)
+		(pin "C6"
+		)
+		(pin "H1"
+		)
+		(pin "D3"
+		)
+		(pin "E4"
+		)
+		(pin "D6"
+		)
+		(pin "C7"
+		)
+		(pin "H7"
+		)
+		(pin "C2"
+		)
+		(pin "B5"
+		)
+		(pin "C5"
+		)
+		(pin "G2"
+		)
+		(pin "G6"
+		)
+		(pin "A7"
+		)
+		(pin "E2"
+		)
+		(pin "E7"
+		)
+		(pin "G7"
+		)
+		(pin "F2"
+		)
+		(pin "H2"
+		)
+		(pin "B6"
+		)
+		(pin "E5"
+		)
+		(pin "G1"
+		)
+		(pin "A5"
+		)
+		(pin "E1"
+		)
+		(pin "F6"
+		)
+		(pin "C1"
+		)
+		(pin "C3"
+		)
+		(pin "D1"
+		)
+		(pin "B2"
+		)
+		(pin "G4"
+		)
+		(pin "H6"
+		)
+		(pin "B7"
+		)
+		(pin "A1"
+		)
+		(pin "D4"
+		)
+		(pin "B4"
+		)
+		(pin "F4"
+		)
+		(pin "F3"
+		)
+		(pin "A4"
+		)
+		(pin "A3"
+		)
+		(pin "A6"
+		)
+		(pin "B3"
+		)
+		(pin "B1"
+		)
+		(instances
+			(project "projector"
+				(path "/0c7b44f4-2a5d-4ccb-91ae-fa3b66550b5b"
+					(reference "U1")
+					(unit 1)
+				)
+			)
+		)
+	)
 	(sheet_instances
 		(path "/"

Commit message: Improve DLPA2000 symbol
Parts:
- added U2: DLPC1438, litho:NFBGA201, symbol litho:DLPC1438
- added U3: DLP301S, litho:INTERPOSER_TODO, symbol litho:DLP301S
- U1: footprint YFF56_TEX -> custom_dlp:YFF56_TEX
Connections:
- new net: U2.C2 (DD3N), U2.F3 (RREF)
- new net VBIAS: U3.A22 (VBIAS), U3.A6 (VBIAS)
- new net VCC18: U2.C7 (VCC18), U2.C9 (VCC18), U2.D4 (VCC18), U2.E12 (VCC18), U2.F12 (VCC18), U2.K13 (VCC18), U2.M11 (VCC18)
- new net VCC_INTF: U2.M3 (VCC_INTF), U2.M7 (VCC_INTF), U2.N3 (VCC_INTF), U2.N7 (VCC_INTF)
- new net VDD: U2.C5 (VDD), U2.D12 (VDD), U2.D13 (VDD), U2.D3 (VDD), U2.D5 (VDD), U2.D7 (VDD), U2.D9 (VDD), U2.E3 (VDD), U2.F13 (VDD), U2.H13 (VDD), U2.J12 (VDD), U2.J4 (VDD), U2.K3 (VDD), U2.L12 (VDD), U2.L13 (VDD), U2.L4 (VDD), U2.M10 (VDD), U2.M6 (VDD), U2.M9 (VDD), U3.A19 (VDD), U3.A20 (VDD), U3.A21 (VDD), U3.B20 (VDD), U3.C2 (VDD), U3.D2 (VDD), U3.D23 (VDD), U3.D3 (VDD), U3.E2 (VDD), U3.F2 (VDD), U3.F23 (VDD), U3.F3 (VDD)
- new net VDDI: U3.B19 (VDDI), U3.B6 (VDDI), U3.C23 (VDDI), U3.C3 (VDDI), U3.E23 (VDDI), U3.E3 (VDDI), U3.G23 (VDDI), U3.G3 (VDDI)
- new net VOFFSET: U3.B21 (VOFFSET), U3.G2 (VOFFSET)
- new net VRESET: U3.A23 (VRESET), U3.A5 (VRESET)
- new net VSS: U2.C4 (VSS), U2.C6 (VSS), U2.C8 (VSS), U2.D10 (VSS), U2.D6 (VSS), U2.D8 (VSS), U2.E13 (VSS), U2.E4 (VSS), U2.F10 (VSS), U2.F4 (VSS), U2.F6 (VSS), U2.F7 (VSS), U2.F8 (VSS), U2.F9 (VSS), U2.G10 (VSS), U2.G12 (VSS), U2.G13 (VSS), U2.G4 (VSS), U2.G6 (VSS), U2.G7 (VSS), U2.G8 (VSS), U2.G9 (VSS), U2.H10 (VSS), U2.H12 (VSS), U2.H4 (VSS), U2.H6 (VSS), U2.H7 (VSS), U2.H8 (VSS), U2.H9 (VSS), U2.J10 (VSS), U2.J13 (VSS), U2.J3 (VSS), U2.J6 (VSS), U2.J7 (VSS), U2.J8 (VSS), U2.J9 (VSS), U2.K10 (VSS), U2.K12 (VSS), U2.K4 (VSS), U2.K6 (VSS), U2.K7 (VSS), U2.K8 (VSS), U2.K9 (VSS), U2.L3 (VSS), U2.M12 (VSS), U2.M4 (VSS), U2.M5 (VSS), U2.M8 (VSS), U3.A2 (VSS), U3.A24 (VSS), U3.A3 (VSS), U3.A4 (VSS), U3.A7 (VSS), U3.B22 (VSS), U3.B23 (VSS), U3.B24 (VSS), U3.C19 (VSS), U3.C22 (VSS), U3.C4 (VSS), U3.C7 (VSS), U3.E19 (VSS), U3.E22 (VSS), U3.E4 (VSS), U3.E7 (VSS), U3.G19 (VSS), U3.G22 (VSS), U3.G24 (VSS), U3.G4 (VSS), U3.G7 (VSS), U3.H2 (VSS), U3.H23 (VSS), U3.H24 (VSS), U3.H3 (VSS)

Commit message: Partial work on PMIC
Parts:
- removed U1: DLPA2000DYFFR, custom_dlp:YFF56_TEX, symbol litho:DLPA2000DYFFR
- removed unit 2 of U2
- removed unit 8 of U2
- removed unit 6 of U2
- removed unit 3 of U2
- removed unit 4 of U2
- added C1: 1uF, symbol Device:C
- added C10, C11, C12, C9: 22uF, symbol Device:C
- added C2, C3, C5: 10uF, symbol Device:C
- added C4: 20uF, symbol Device:C
- added C6, C7: 0.1uF, symbol Device:C
- added C8: 2.2uF, symbol Device:C
- added J2: To LED, symbol Connector:Conn_01x04_Pin
- added L1: 2.2uH, RSL48_4P4X4P4_TEX, symbol Device:L
- added U1: DLPA2005ERSLR, RSL48_4P4X4P4_TEX, symbol litho:DLPA2005ERSLR
- J1: renamed from U3; value DLP301S -> To DLP301S
Connections:
- net at U2.B14 (LED_SEL_1): now also U1.34 (LED_SEL1)
- net at U2.B15 (LED_SEL_0): now also U1.31 (LED_SEL0)
- net at U2.C14 (GPIO_00/SPI1_DIN): now also U1.3 (SPI_DIN)
- net at U2.C15 (GPIO_01/SPI1_CLK): now also U1.7 (SPI_CLK)
- net at U2.D14 (GPIO_02/SPI1_DOUT): now also U1.9 (SPI_DOUT)
- new net: C8.2, U1.19 (V2V5)
- new net: C7.2, U1.35 (V6V)
- new net: L1.1, U1.47 (L1), U1.48 (L1)
- new net: L1.2, U1.43 (L2), U1.44 (L2)
- new net: C6.2, U1.32 (VSPI)
- new net +5V: C1.1, C2.1, C3.1, C4.1, C5.2, U1.1 (VINL), U1.10 (VINR), U1.2 (VINL)
- new net GND: C1.2, C10.1, C11.1, C12.1, C2.2, C3.2, C4.2, C5.1, C6.1, C7.1, C8.1, C9.1, U1.12 (PGNDR), U1.20 (GND), U1.23 (PGNDC), U1.45 (PGNDL), U1.46 (PGNDL), U1.49 (EPAD), U1.5 (AGND1)
- new net LED_ANODE: C10.2, C11.2, C12.2, C9.2, J2.4 (Pin_4), U1.41 (VLED), U1.42 (VLED)
- new net RED_CATHODE: J2.3 (Pin_3), U1.39 (SW4)
- new net UNUSED_CONN: J2.2 (Pin_2), U1.38 (SW5)
- new net UV_CATHODE: J2.1 (Pin_1), U1.37 (SW6)
Other:
- note added: "Connect thermal vias to GND plane"
- note added: "DLP301S on interposer connected via ribbon cable"
- note added: "DMD INTERFACE"
- note added: "Noisy SMPS. Place away from data lines."
- note added: "SMPS GND"
- note added: "TODO: See what to do with GPIO_04"
- note added: "This board expects +5 V input and uses the DLPA2005 to regulate down to the lower values needed for operation GND should be a full ground plane in a 4 layer board. Place bypass caps as close as possible to designated pin"
- note added: "~5A"
- moved on the sheet: J1, U2E, U2G

Commit message: More projector power supply design
Parts:
- added D1: HSMG-C170, Diode_SMD:D_0805_2012Metric_Pad1.15x1.40mm_HandSolder, symbol Device:LED
- added R1: 39m, 3 W, Resistor_SMD:R_2512_6332Metric_Pad1.40x3.35mm_HandSolder, symbol Device:R
- added R2: 510, Resistor_SMD:R_0805_2012Metric_Pad1.20x1.40mm_HandSolder, symbol Device:R
- C1: footprint (none) -> Capacitor_SMD:C_0603_1608Metric_Pad1.08x0.95mm_HandSolder; Digikey (none) -> 1276-1946-1-ND
- C10, C11, C12, C9: footprint (none) -> Capacitor_THT:CP_Radial_D5.0mm_P2.00mm; Digikey (none) -> 732-8789-1-ND
- C2, C3, C5: footprint (none) -> Capacitor_SMD:C_0805_2012Metric_Pad1.18x1.45mm_HandSolder; Digikey (none) -> 490-3886-1-ND
- C4: value 20uF -> 22uF; footprint (none) -> Capacitor_THT:CP_Radial_D5.0mm_P2.00mm; Digikey (none) -> 732-8789-1-ND
- L1: footprint RSL48_4P4X4P4_TEX -> (none)
- U1, U2: Digikey (none) -> ORDER FROM TI
Connections:
- net +5V: now also D1.2 (A)
- net GND: now also R1.2, R2.2
- net at U1.36 (RLIM_K): now also U1.40 (RLIM), R1.1
- new net: D1.1 (K), R2.1
Other:
- note added: "Connect RLIM_K with it's own trace consult datasheet for details."
- note added: "Noisy SMPS. Place away from data lines. Keep inductor loops small"
- note added: "Power Indicator LEDs"
- note added: "SPI 33.3 MHz Max"
- note added: "This board expects +5 V input and uses the DLPA2005 to regulate up/down to the values needed for operation GND should be a full ground plane in a 4 layer board. Place bypass caps as close as possible to designated pin General TODOS: Select Micro, Talk to rest of the group about +5V source. Decide on HMI"
- note added: "f_sw = 2.25 MHz"
- note added: "~3 A"
- note added: "~5A, +5V"
- note removed: "Noisy SMPS. Place away from data lines."
- note removed: "This board expects +5 V input and uses the DLPA2005 to regulate down to the lower values needed for operation GND should be a full ground plane in a 4 layer board. Place bypass caps as close as possible to designated pin"
- note removed: "~5A"
- company: (none) -> MICHIGAN TECH OPEN SOURCE HARDWARE ENTERPRISE
- title: (none) -> LITHO_PROJECTOR
- moved on the sheet: C1, C10, C11, C12, C2, C3, C4, C5, C6, C7, C8, C9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

Commit message: Add more stuff
Parts:
- added C13, C14, C15: 47uF, Capacitor_THT:CP_Radial_D5.0mm_P2.00mm, symbol Device:C_Polarized
- added D2, D3, D4: HSMG-C170, Diode_SMD:D_0805_2012Metric_Pad1.15x1.40mm_HandSolder, symbol Device:LED
- added J3: To PWR, symbol Connector:Conn_01x04_Pin
- added R3, R4, R5: 100k, symbol Device:R
- added R6, R7, R8: 510, Resistor_SMD:R_0805_2012Metric_Pad1.20x1.40mm_HandSolder, symbol Device:R
- C4: symbol Device:C -> Device:C_Polarized
Connections:
- net +5V: now also C13.1, J3.1 (Pin_1)
- net GND: now also C13.2, C14.2, C15.2, J3.4 (Pin_4), R6.2, R7.2, R8.2
- net at U1.3 (SPI_DIN): no longer U2.C14 (GPIO_00/SPI1_DIN)
- net at U1.7 (SPI_CLK): no longer U2.C15 (GPIO_01/SPI1_CLK)
- net at U1.9 (SPI_DOUT): no longer U2.D14 (GPIO_02/SPI1_DOUT)
- net at U2.D15 (GPIO_03/SPI1_CSZ0): now also R3.2
- new net: D3.1 (K), R7.1
- new net: D4.1 (K), R8.1
- new net: D2.1 (K), R6.1
- new net: R5.2, U2.C15 (GPIO_01/SPI1_CLK)
- new net: R4.2, U2.D14 (GPIO_02/SPI1_DOUT)
- new net +1V8_SRC: C15.1, D3.2 (A), J3.3 (Pin_3)
- new net +1V8_SW: D4.2 (A), R3.1, R4.1, R5.1
- new net +3V3: C14.1, D2.2 (A), J3.2 (Pin_2)
Other:
- note added: "SPI Max Freq: 33.3 MHz"
- note added: "TODO: Check if correct 1.8V supply"
- note added: "This board expects +5 V input and uses the DLPA2005 to regulate up/down to the values needed for operation. It may draw up to 5 A of current but will likely be less than that in normal operation GND should be a full ground plane in a 4 layer board. Place bypass caps as close as possible to designated pin General TODOS: Select Micro, Talk to rest of the group about +5V source. Decide on HMI"
- note added: "f_sw = 2.25 MHz 4 A max"
- note removed: "SPI 33.3 MHz Max"
- note removed: "TODO: See what to do with GPIO_04"
- note removed: "This board expects +5 V input and uses the DLPA2005 to regulate up/down to the values needed for operation GND should be a full ground plane in a 4 layer board. Place bypass caps as close as possible to designated pin General TODOS: Select Micro, Talk to rest of the group about +5V source. Decide on HMI"
- note removed: "f_sw = 2.25 MHz"
- moved on the sheet: D1, R2

Commit message: Added resistor.
Parts:
- C6, C7: footprint (none) -> Capacitor_SMD:C_0603_1608Metric_Pad1.08x0.95mm_HandSolder; Digikey (none) -> 4713-GMC10X7R104K50NTCT-ND
Changed lines of the file:
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@@
 			)
 		)
-		(property "Footprint" ""
+		(property "Footprint" "Capacitor_SMD:C_0603_1608Metric_Pad1.08x0.95mm_HandSolder"
 			(at 241.6048 53.34 0)
 			(hide yes)
@@
 		)
 		(property "Description" "Unpolarized capacitor"
+			(at 242.57 57.15 0)
+			(hide yes)
+			(show_name no)
+			(do_not_autoplace no)
+			(effects
+				(font
+					(size 1.27 1.27)
+				)
+			)
+		)
+		(property "Digikey" "4713-GMC10X7R104K50NTCT-ND"
 			(at 242.57 57.15 0)
 			(hide yes)
@@
 			)
 		)
-		(property "Footprint" ""
+		(property "Footprint" "Capacitor_SMD:C_0603_1608Metric_Pad1.08x0.95mm_HandSolder"
 			(at 143.51 82.8548 0)
 			(hide yes)
@@
 			(hide yes)
 			(show_name no)
+			(do_not_autoplace no)
+			(effects
+				(font
+					(size 1.27 1.27)
+				)
+			)
+		)
+		(property "Digikey" "4713-GMC10X7R104K50NTCT-ND"
+			(at 139.7 83.82 90)
+			(hide yes)
+			(show_name no)

Commit message: Finish SPI bus
Parts:
- added R10, R11, R12, R9: 30.1, symbol Device:R
Connections:
- net +1V8_SW: now also C6.2, U1.32 (VSPI)
- net at R3.2: now also U1.8 (SPI_CSZ), R12.2; no longer U2.D15 (GPIO_03/SPI1_CSZ0)
- net at U1.3 (SPI_DIN): now also R4.2, R9.2
- net at U1.7 (SPI_CLK): now also R5.2, R11.2
- net at U1.9 (SPI_DOUT): now also R10.2
- net at U2.C14 (GPIO_00/SPI1_DIN): now also R10.1
- net at U2.C15 (GPIO_01/SPI1_CLK): now also R11.1; no longer R5.2
- net at U2.D14 (GPIO_02/SPI1_DOUT): now also R9.1; no longer R4.2
- new net: R12.1, U2.D15 (GPIO_03/SPI1_CSZ0)
Other:
- note added: "Probably does not need to be impedence matched, See: https://resources.altium.com/p/there-spi-trace-impedance-requirement"
- note added: "TODO: Check low voltage indicators have low enough resistor"
- note added: "This board requires 3 external power supplies: +5V 4.5A, +3.3V 1A, +1.8V 0.5A GND should be a full ground plane in a 4 layer board. Place bypass caps as close as possible to designated pin General TODOS: Select Micro. Decide on HMI"
- note removed: "This board expects +5 V input and uses the DLPA2005 to regulate up/down to the values needed for operation. It may draw up to 5 A of current but will likely be less than that in normal operation GND should be a full ground plane in a 4 layer board. Place bypass caps as close as possible to designated pin General TODOS: Select Micro, Talk to rest of the group about +5V source. Decide on HMI"
- moved on the sheet: C13, C14, C15, C6, D1, D2, D3, D4, J1, J3, R2, R6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

Commit message: More projector power work
Parts:
- removed D3, D4: HSMG-C170, Diode_SMD:D_0805_2012Metric_Pad1.15x1.40mm_HandSolder, symbol Device:LED
- removed R7, R8: 510, Resistor_SMD:R_0805_2012Metric_Pad1.20x1.40mm_HandSolder, symbol Device:R
- added C16: 2.2uF, symbol Device:C
- added C17: 1uF, Capacitor_SMD:C_0603_1608Metric_Pad1.08x0.95mm_HandSolder, symbol Device:C
- added C18: 10uF, Capacitor_SMD:C_0805_2012Metric_Pad1.18x1.45mm_HandSolder, symbol Device:C
- added C19: 0.1uF, Capacitor_SMD:C_0603_1608Metric_Pad1.08x0.95mm_HandSolder, symbol Device:C
- added L2: 2.2uH, Inductor_SMD:L_1008_2520Metric_Pad1.43x2.20mm_HandSolder, symbol Device:L
- added R13: 10k, symbol Device:R
- added R14: DNP, Resistor_SMD:R_0603_1608Metric, symbol Device:R
- added TP1: 1V8_SRC, TestPoint:TestPoint_Pad_2.0x2.0mm, symbol Connector:TestPoint
- added TP2: 1V8_SW, TestPoint:TestPoint_Pad_2.0x2.0mm, symbol Connector:TestPoint
- added TP3, TP4: GND, TestPoint:TestPoint_Pad_2.0x2.0mm, symbol Connector:TestPoint
- added TP5: VCORE, TestPoint:TestPoint_Pad_2.0x2.0mm, symbol Connector:TestPoint
- added TP6: +6V, TestPoint:TestPoint_Pad_2.0x2.0mm, symbol Connector:TestPoint
- added TP7: +2V5, TestPoint:TestPoint_Pad_2.0x2.0mm, symbol Connector:TestPoint
- added TP8: VLED, TestPoint:TestPoint_Pad_2.0x2.0mm, symbol Connector:TestPoint
Connections:
- net +1V8_SRC: now also TP1.1
- net +1V8_SW: now also R13.1, R14.1, TP2.1
- net +3V3: now also U1.25 (VINC), C16.2
- net +5V: now also U1.18 (VINA), C17.1, C19.2
- net GND: now also C16.1, C17.2, C18.2, C19.1, TP3.1, TP4.1
- net LED_ANODE: now also TP8.1
- net at C8.2, U1.19 (V2V5): now also TP7.1
- net at C7.2, U1.35 (V6V): now also TP6.1
- net RESETZ: now reaches U2.C11 (RESETZ)
- net RESETZ: now also U1.4 (RESETZ), R14.2
- net INTZ: now reaches U2.C13 (PARKZ)
- net INTZ: now also U1.6 (INTZ), R13.2
- net at U1.24 (SWC): now also L2.2
- net PROJ_ON: now reaches U1.27 (PROJ_ON)
- net +VCORE: now reaches U1.29 (VCORE)
- net +VCORE: now also C18.1, L2.1, TP5.1
Other:
- note added: "1.8V is not enough to bias most cheap LEDs"
- note added: "Power Indicator"
- note removed: "Power Indicator LEDs"
- note removed: "TODO: Check low voltage indicators have low enough resistor"
- moved on the sheet: C1, C2, C3, C4, C5, U2A
