File: micromanipulator-board/umanip.kicad_sch (KiCad schematic)
At the start: 0 parts

Commit message: Revision 1 Micromanipulator
Started Design
Parts:
- added A1: RaspberryPi_Pico, Module:RaspberryPi_Pico_Common_Unspecified, symbol MCU_Module:RaspberryPi_Pico
- added C1: 2.2uF, symbol Device:C
- added C13, C14: 47uF, Capacitor_THT:CP_Radial_D5.0mm_P2.00mm, symbol Device:C_Polarized
- added D1, D2: HSMG-C170, Diode_SMD:D_0805_2012Metric_Pad1.15x1.40mm_HandSolder, symbol Device:LED
- added J1, J2, J3, J4, J5: Conn_01x04_Pin, symbol Connector:Conn_01x04_Pin
- added R1: 10k, symbol Device:R
- added R2, R3: 510, Resistor_SMD:R_0805_2012Metric_Pad1.20x1.40mm_HandSolder, symbol Device:R
Connections:
- new net: D2.1 (K), R3.1
- new net: D1.1 (K), R2.1
- new net +12V: C13.1, D2.2 (A), J5.1 (Pin_1)
- new net +3.3V: A1.39 (VSYS), C14.1, D1.2 (A), J5.2 (Pin_2), R1.1
- new net Diag1: A1.5 (GPIO3)
- new net Diag2: A1.10 (GPIO7)
- new net Diag3: A1.15 (GPIO11)
- new net Diag4: A1.20 (GPIO15)
- new net Dir1: A1.1 (GPIO0)
- new net Dir2: A1.6 (GPIO4)
- new net Dir3: A1.11 (GPIO8)
- new net Dir4: A1.16 (GPIO12)
- new net EN1: A1.4 (GPIO2)
- new net EN2: A1.9 (GPIO6)
- new net EN3: A1.14 (GPIO10)
- new net EN4: A1.19 (GPIO14)
- new net GND: A1.13 (GND), A1.18 (GND), A1.23 (GND), A1.28 (GND), A1.3 (GND), A1.38 (GND), A1.8 (GND), C13.2, C14.2, J5.4 (Pin_4), R1.2, R2.2, R3.2
- new net RX: A1.21 (GPIO16)
- new net Step1: A1.2 (GPIO1)
- new net Step2: A1.7 (GPIO5)
- new net Step3: A1.12 (GPIO9)
- new net Step4: A1.17 (GPIO13)
- new net TX: A1.22 (GPIO17)
Other:
- note added: "CHANGE TO HAND SOLDERABLE AND LIGHT TYPE SO DOESN'T AFFECT UV"
- note added: "Can do 5V instead of 3.3V for microcontroller too**"
- note added: "Power Indicator Lights"
- note added: "Stepper 1 (X1)"
- note added: "Stepper 2 (X2)"
- note added: "Stepper 3 (Y)"
- note added: "Stepper 4 (Z)"
- note added: "Stepper Motors Are NEMA 17"
- note added: "The Pico 2 digital pins tolerate 5V logic when powered with 3.3V"

Commit message: Micromanipulator Documentation
Uart Labels and Etc
Parts:
- R1: footprint (none) -> Resistor_THT:R_Axial_DIN0207_L6.3mm_D2.5mm_P10.16mm_Horizontal
Connections:
- net GND: no longer A1.13 (GND), A1.18 (GND), A1.23 (GND), A1.28 (GND), A1.3 (GND), A1.38 (GND), A1.8 (GND)
- new net: A1.13 (GND), A1.18 (GND), A1.23 (GND), A1.28 (GND), A1.3 (GND), A1.38 (GND), A1.8 (GND)
Other:
- note added: "CHECK DATA SHEET - DECOUPLE +12V FEED @ DRIVER"
- note added: "UART ADDRESS REFERENCES: Stepper 1 (X1) M1- Low (0) M2- Low (0) Stepper 2 (X2) M1- Low (0) M2- High (1) Stepper 3 (Y) M1- High (1) M2- Low (0) Stepper 4 (Z) M1- High (1) M2- High (1)"
- company: (none) -> MICHIGAN TECH OPEN SOURCE HARDWARE ENTERPRISE
- title: (none) -> Micro Manipulator
- moved on the sheet: A1, C1, J1, J2, J3, J4, R1
